File: reverie.kicad_pcb (KiCad board)
At the start: 2 copper layers, 334.4 x 81.5 mm, 141 parts, among them SW1 SW_Push, U1 PRTR5V0U2X, U2 ATmega32U4-AU, Y1 16MHz

Commit message: initial layout and routing
Parts:
- removed R5, R6: 22, Resistor_SMD:R_0805_2012Metric
- C1, C2: value 22uF -> 22pF
- moved SW1 80.6 mm to (78.4, 122.9)
- moved C7 80.5 mm to (58.4, 115.1)
- moved R8 68.1 mm to (71.6, 110.9), turned to 180 degrees
- moved C4 67.8 mm to (71.1, 102.4), turned to 90 degrees
- moved R1 66.4 mm to (71.5, 115.2)
- moved C5 65.6 mm to (65.5, 115.1), turned to 180 degrees
- moved C6 63.7 mm to (53.7, 101.0), turned to 180 degrees
- moved C3 61.3 mm to (50.2, 106.2), turned to 180 degrees
- moved C2 61.1 mm to (65.9, 94.9), turned to 90 degrees
- moved C1 55.9 mm to (58.9, 94.9), turned to 270 degrees
- moved Y1 53.1 mm to (62.5, 94.9)
- moved R4 52.8 mm to (50.2, 108.2), turned to 180 degrees
- moved R3 51.8 mm to (50.2, 110.2), turned to 180 degrees
- moved R7 33.1 mm to (51.8, 79.4), turned to 90 degrees
- moved U1 25.9 mm to (74.4, 76.5), turned to 180 degrees
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Connections:
- F1 pad 1: VCC -> +5V
- R1 pad 2: Net-(R1-Pad2) -> +5V
- U1 pad 1: Net-(U1-Pad1) -> GND
- U2 pad 14: Net-(R1-Pad2) -> +5V
- U2 pad 2: Net-(R1-Pad2) -> +5V
- U2 pad 24: Net-(R1-Pad2) -> +5V
- U2 pad 3: Net-(R6-Pad1) -> D-
- U2 pad 34: Net-(R1-Pad2) -> +5V
- U2 pad 4: Net-(R5-Pad1) -> D+
- U2 pad 44: Net-(R1-Pad2) -> +5V
Routing:
- net ROW2: track 0.00 -> 418.0 mm, vias 0 -> 16
- net ROW3: track 0.00 -> 405.0 mm, vias 0 -> 1
- net ROW1: track 0.00 -> 389.8 mm, vias 0 -> 15
- net ROW0: track 0.00 -> 345.4 mm, vias 0 -> 16
- net COL15: track 0.00 -> 284.6 mm, vias 0 -> 1
- net COL16: track 0.00 -> 272.9 mm, vias 0 -> 1
- net COL14: track 0.00 -> 258.9 mm, vias 0 -> 1
- net COL12: track 0.00 -> 223.2 mm, vias 0 -> 1
- net COL13: track 0.00 -> 220.8 mm, vias 0 -> 1
- net COL10: track 0.00 -> 187.0 mm, vias 0 -> 1
- net COL11: track 0.00 -> 183.3 mm, vias 0 -> 1
- net COL9: track 0.00 -> 145.9 mm, vias 0 -> 1
- net COL7: track 0.00 -> 138.7 mm, vias 0 -> 1
- net COL0: track 0.00 -> 134.0 mm, vias 0 -> 1
- net COL8: track 0.00 -> 125.8 mm, vias 0 -> 1
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- added copper zone on B.Cu, net GND
- added copper zone on F.Cu, net GND
Other:
- board size 334.4 x 81.5 mm -> 333.4 x 88.7 mm
- net class Default: trace_width 0.25 -> 0.254
- net class Power added: clearance 0.2, trace_width 0.381, via_dia 0.8, via_drill 0.4

Commit message: complete routing
add ISP programmer
Parts:
- moved C5 1.94 mm to (67.4, 114.7)
- moved C7 1.80 mm to (56.6, 115.3)
- moved C4 1.33 mm to (71.5, 101.1)
- moved C6 1.28 mm to (52.5, 100.8)
- moved R1 0.92 mm to (72.3, 114.7)
- moved R8 0.74 mm to (72.0, 111.5)
Connections:
- U2 pad 36: Net-(U2-Pad36) -> COL12
- U2 pad 37: Net-(U2-Pad37) -> COL11
- U2 pad 38: Net-(U2-Pad38) -> COL10
- U2 pad 39: Net-(U2-Pad39) -> COL9
- U2 pad 40: Net-(U2-Pad40) -> COL8
- U2 pad 41: Net-(U2-Pad41) -> COL7
Routing:
- net ROW1: track 389.8 -> 438.5 mm, vias 15 -> 16
- net ROW3: track 405.0 -> 443.8 mm, vias 1 -> 2
- net ROW2: track 418.0 -> 455.4 mm, vias 16 -> 17
- net COL7: track 138.7 -> 167.8 mm, vias 1 -> 2
- net COL8: track 125.8 -> 153.5 mm, vias 1 -> 2
- net COL9: track 145.9 -> 172.0 mm, vias 1 -> 2
- net COL10: track 187.0 -> 212.7 mm, vias 1 -> 2
- net COL11: track 183.3 -> 207.2 mm, vias 1 -> 2
- net COL12: track 223.2 -> 245.9 mm, vias 1 -> 2
- net ROW0: track 345.4 -> 367.5 mm, vias 16 -> 17
- net +5V: track 93.6 -> 110.7 mm
- net COL0: track 134.0 -> 149.4 mm, vias 1 -> 2
- net COL1: track 114.5 -> 130.0 mm, vias 1 -> 2
- net COL5: track 96.4 -> 110.9 mm, vias 1 -> 2
- net COL4: track 78.4 -> 92.9 mm, vias 1 -> 2
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
Commit message: clean up
Parts:
- added J1: AVR-ISP-6, Connector_IDC:IDC-Header_2x03_P2.54mm_Vertical, F.Cu at (49.0, 96.3)
- MX56: footprint MX_Only:MXOnly-2.25U-Hotswap -> MX_Only:MXOnly-2.25U-Hotswap-ReversedStabilizers
- MX57: footprint MX_Only:MXOnly-2.75U-Hotswap -> MX_Only:MXOnly-2.75U-Hotswap-ReversedStabilizers
- moved C6 1.65 mm to (50.8, 100.8)
Connections:
- net Net-(R1-Pad1) renamed RST
- U2 pad 10: Net-(U2-Pad10) -> MOSI
- U2 pad 11: Net-(U2-Pad11) -> MISO
- U2 pad 12: Net-(U2-Pad12) -> ROW1
- U2 pad 18: Net-(U2-Pad18) -> ROW2
- U2 pad 19: Net-(U2-Pad19) -> ROW3
- U2 pad 20: Net-(U2-Pad20) -> COL2
- U2 pad 21: Net-(U2-Pad21) -> COL1
- U2 pad 22: Net-(U2-Pad22) -> COL0
- U2 pad 25: Net-(U2-Pad25) -> ROW0
- U2 pad 26: Net-(U2-Pad26) -> COL5
- U2 pad 27: Net-(U2-Pad27) -> COL4
- U2 pad 28: Net-(U2-Pad28) -> COL6
- U2 pad 29: Net-(U2-Pad29) -> COL16
- U2 pad 30: Net-(U2-Pad30) -> COL15
- U2 pad 31: Net-(U2-Pad31) -> COL14
- U2 pad 32: Net-(U2-Pad32) -> COL13
- U2 pad 8: Net-(U2-Pad8) -> COL3
- U2 pad 9: Net-(U2-Pad9) -> SCK
Routing:
- net MOSI: track 0.00 -> 20.6 mm, vias 0 -> 1
- net MISO: track 0.00 -> 12.2 mm, vias 0 -> 2
- net +5V: track 110.7 -> 122.5 mm
- net SCK: track 0.00 -> 11.3 mm, vias 0 -> 1
- net GND: track 47.0 -> 56.4 mm, vias 10 -> 14
- net RST: track 31.6 -> 40.9 mm, vias 2 -> 3
- net COL2: track 110.5 -> 118.7 mm
- net ROW2: track 455.4 -> 459.3 mm
- net COL3: track 66.7 -> 69.9 mm
- net COL6: track 117.1 -> 119.4 mm
- net Net-(R4-Pad2): track 61.1 -> 63.2 mm
- net COL1: track 130.0 -> 131.3 mm
- net ROW3: track 443.8 -> 445.0 mm
- net COL5: track 110.9 -> 112.1 mm
- net COL0: track 149.4 -> 150.6 mm
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Other:
- outline, holes or cut-outs redrawn

Commit message: add vanity silk text
Other:
- board text added: "REVERIE_V0 BY MAKENOVA"
Changed lines of the file:
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@@
   (general
     (thickness 1.6)
-    (drawings 11)
+    (drawings 12)
     (tracks 1234)
     (zones 0)
@@
     )
   )
+  (gr_text "REVERIE_V0\n\nBY MAKENOVA" (at 63.246 112.649) (layer F.SilkS)
+    (effects (font (size 3 3) (thickness 0.3)))
+  )
   (gr_line (start 69.604454 73.078101) (end 69.75841 73.09582) (layer Edge.Cuts) (width 0.2))

Commit message: reshape edge cuts
regenerate gerber drill files and tracespace
Routing:
- net GND: vias 14 -> 17
Other:
- board size 333.4 x 88.7 mm -> 333.4 x 88.8 mm
Changed lines of the file:
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@@
   (general
     (thickness 1.6)
-    (drawings 12)
-    (tracks 1234)
+    (drawings 16)
+    (tracks 1237)
     (zones 0)
     (modules 140)
@@
     (visible_elements FFFFFF7F)
     (pcbplotparams
-      (layerselection 0x010fc_ffffffff)
+      (layerselection 0x010f0_ffffffff)
       (usegerberextensions false)
       (usegerberattributes false)
@@
       (outputformat 1)
       (mirror false)
-      (drillshape 1)
+      (drillshape 0)
       (scaleselection 1)
-      (outputdirectory ""))
+      (outputdirectory "gerber/"))
   )
   (net 0 "")
@@
     )
   )
+  (gr_line (start 324.485 149.352) (end 324.477 73.16) (layer Edge.Cuts) (width 0.2))
+  (gr_line (start -8.89 149.479) (end -8.898 73.16) (layer Edge.Cuts) (width 0.2))
+  (gr_line (start 95.758 149.479) (end 324.485 149.352) (layer Edge.Cuts) (width 0.2))
+  (gr_line (start 29.464 149.479) (end -8.89 149.479) (layer Edge.Cuts) (width 0.2))
+  (gr_line (start 34.036 154.051) (end 91.059 154.178) (layer Edge.Cuts) (width 0.2))
+  (gr_arc (start 34.036 149.479) (end 29.464 149.479) (angle -90) (layer Edge.Cuts) (width 0.2))
+  (gr_arc (start 91.059 149.479) (end 91.059 154.178) (angle -90) (layer Edge.Cuts) (width 0.2))
   (gr_text "REVERIE_V0\n\nBY MAKENOVA" (at 63.246 112.649) (layer F.SilkS)
     (effects (font (size 3 3) (thickness 0.3)))
@@
   (gr_line (start 67.691 71.02841) (end 67.691 65.405) (layer Edge.Cuts) (width 0.2))
   (gr_line (start 57.277 65.405) (end 67.691 65.405) (layer Edge.Cuts) (width 0.2))
-  (gr_line (start 324.477 73.16) (end 324.477 154.1225) (layer Edge.Cuts) (width 0.2))
-  (gr_line (start -8.898 73.16) (end -8.898 154.1225) (layer Edge.Cuts) (width 0.2))
-  (gr_line (start -8.898 154.1225) (end 324.477 154.1225) (layer Edge.Cuts) (width 0.2))
   (segment (start 59.259 72.01) (end 58.164 70.915) (width 0.381) (layer B.Cu) (net 1))
   (segment (start 59.259 72.33) (end 59.259 72.01) (width 0.381) (layer B.Cu) (net 1))
@@
   (via (at 52.959 92.583) (size 0.8) (drill 0.4) (layers F.Cu B.Cu) (net 1))
   (segment (start 54.102 93.726) (end 52.959 92.583) (width 0.381) (layer B.Cu) (net 1))
+  (via (at 193.675 146.812) (size 0.8) (drill 0.4) (layers F.Cu B.Cu) (net 1))
+  (via (at 221.107 147.066) (size 0.8) (drill 0.4) (layers F.Cu B.Cu) (net 1))
+  (via (at 199.136 136.779) (size 0.8) (drill 0.4) (layers F.Cu B.Cu) (net 1))
   (segment (start 61.2965 93.9315) (end 61.384 94.019) (width 0.254) (layer B.Cu) (net 2))
   (segment (start 58.928 93.9315) (end 61.2965 93.9315) (width 0.254) (layer B.Cu) (net 2))
@@
   (segment (start 51.816 150.875) (end 70.866 150.875) (width 0.254) (layer B.Cu) (net 58))
   (segment (start 70.866 150.875) (end 89.789 150.875) (width 0.254) (layer B.Cu) (net 58))
-  (segment (start 118.364 146.88) (end 118.364 146.176) (width 0.254) (layer B.Cu) (net 58))
-  (segment (start 114.369 150.875) (end 118.364 146.88) (width 0.254) (layer B.Cu) (net 58))
-  (segment (start 89.789 150.875) (end 114.369 150.875) (width 0.254) (layer B.Cu) (net 58))
   (segment (start 118.364 146.176) (end 147.066 146.176) (width 0.254) (layer B.Cu) (net 58))
   (segment (start 160.528 143.637) (end 169.672 143.637) (width 0.254) (layer B.Cu) (net 58))
@@
   (segment (start 64.084 99.7752) (end 64.084 100.98) (width 0.254) (layer B.Cu) (net 58))
   (segment (start 64.0861 99.7731) (end 64.084 99.7752) (width 0.254) (layer B.Cu) (net 58))
+  (segment (start 91.82 150.875) (end 89.789 150.875) (width 0.254) (layer B.Cu) (net 58))
+  (segment (start 96.519 146.176) (end 91.82 150.875) (width 0.254) (layer B.Cu) (net 58))
+  (segment (start 118.364 146.176) (end 96.519 146.176) (width 0.254) (layer B.Cu) (net 58))
   (segment (start 27.94 140.462) (end 27.94 142.876) (width 0.254) (layer B.Cu) (net 59))
   (segment (start 25.527 138.049) (end 27.94 140.462) (width 0.254) (layer B.Cu) (net 59))
@@
   (segment (start 69.304 107.48) (end 68.184 107.48) (width 0.254) (layer B.Cu) (net 87))
   (segment (start 69.342 107.442) (end 69.304 107.48) (width 0.254) (layer B.Cu) (net 87))
-  (segment (start 75.259 124.786) (end 75.259 123.982) (width 0.254) (layer B.Cu) (net 99))
-  (via (at 59.69 103.378) (size 0.8) (drill 0.4) (layers F.Cu B.Cu) (net 99))
-  (segment (start 59.284 102.972) (end 59.69 103.378) (width 0.254) (layer B.Cu) (net 99))
-  (segment (start 59.284 100.98) (end 59.284 102.972) (width 0.254) (layer B.Cu) (net 99))
-  (segment (start 71.5235 120.2465) (end 71.3255 120.0485) (width 0.254) (layer B.Cu) (net 99))
-  (segment (start 71.3255 120.0485) (end 71.3255 114.681) (width 0.254) (layer B.Cu) (net 99))
-  (segment (start 75.259 123.982) (end 71.5235 120.2465) (width 0.254) (layer B.Cu) (net 99))
-  (via (at 69.977 114.681) (size 0.8) (drill 0.4) (layers F.Cu B.Cu) (net 99))
-  (segment (start 68.961 112.649) (end 69.977 113.665) (width 0.254) (layer F.Cu) (net 99))
-  (segment (start 69.215 112.903) (end 68.961 112.649) (width 0.254) (layer F.Cu) (net 99))
-  (segment (start 68.961 112.649) (end 59.69 103.378) (width 0.254) (layer F.Cu) (net 99))
-  (segment (start 69.977 113.665) (end 69.977 114.681) (width 0.254) (layer F.Cu) (net 99))
-  (segment (start 71.3255 114.681) (end 69.977 114.681) (width 0.254) (layer B.Cu) (net 99))
   (segment (start 52.6565 75.438) (end 49.657 78.4375) (width 0.254) (layer B.Cu) (net 88))
   (segment (start 59.605 75.438) (end 52.6565 75.438) (width 0.254) (layer B.Cu) (net 88))
@@
   (segment (start 70.2455 110.68) (end 71.0715 111.506) (width 0.254) (layer B.Cu) (net 94))
   (segment (start 68.184 110.68) (end 70.2455 110.68) (width 0.254) (layer B.Cu) (net 94))
+  (segment (start 75.259 124.786) (end 75.259 123.982) (width 0.254) (layer B.Cu) (net 99))
+  (via (at 59.69 103.378) (size 0.8) (drill 0.4) (layers F.Cu B.Cu) (net 99))
+  (segment (start 59.284 102.972) (end 59.69 103.378) (width 0.254) (layer B.Cu) (net 99))
+  (segment (start 59.284 100.98) (end 59.284 102.972) (width 0.254) (layer B.Cu) (net 99))
+  (segment (start 71.5235 120.2465) (end 71.3255 120.0485) (width 0.254) (layer B.Cu) (net 99))
+  (segment (start 71.3255 120.0485) (end 71.3255 114.681) (width 0.254) (layer B.Cu) (net 99))
+  (segment (start 75.259 123.982) (end 71.5235 120.2465) (width 0.254) (layer B.Cu) (net 99))
+  (via (at 69.977 114.681) (size 0.8) (drill 0.4) (layers F.Cu B.Cu) (net 99))
+  (segment (start 68.961 112.649) (end 69.977 113.665) (width 0.254) (layer F.Cu) (net 99))
+  (segment (start 69.215 112.903) (end 68.961 112.649) (width 0.254) (layer F.Cu) (net 99))
+  (segment (start 68.961 112.649) (end 59.69 103.378) (width 0.254) (layer F.Cu) (net 99))
+  (segment (start 69.977 113.665) (end 69.977 114.681) (width 0.254) (layer F.Cu) (net 99))
+  (segment (start 71.3255 114.681) (end 69.977 114.681) (width 0.254) (layer B.Cu) (net 99))
   (via (at 54.356 99.2155) (size 0.8) (drill 0.4) (layers F.Cu B.Cu) (net 99))
   (segment (start 58.5235 99.2155) (end 54.356 99.2155) (width 0.254) (layer B.Cu) (net 99))

Commit message: work on edgecuts and replace isp footprint
Parts:
- J1: footprint Connector_IDC:IDC-Header_2x03_P2.54mm_Vertical -> random-keyboard-parts:Reset_Pretty-Mask
- moved J1 2.69 mm to (51.6, 95.4)
- moved D53 2.03 mm to (87.8, 149.2)
Routing:
- net ROW3: track 444.6 -> 446.1 mm
- net MISO: track 12.2 -> 11.7 mm
Other:
- board size 333.4 x 88.8 mm -> 333.4 x 88.6 mm
